File: ISAAC_PCB/ISAAC.sch (KiCad schematic (older format))
At the start: 3 parts

Commit message: Created Schematic
Parts:
- removed Q?: IRF510, TO220, symbol IRF510:IRF510
- added D? (x15): DIODE, Diode_SMD:D_1812_4532Metric_Pad1.30x3.40mm_HandSolder, symbol ISAAC-rescue:DIODE-pspice
- added J? (x2): Screw_Terminal_01x08, TerminalBlock_TE-Connectivity:TerminalBlock_TE_282834-8_1x08_P2.54mm_Horizontal, symbol Connector:Screw_Terminal_01x08
- added R? (x15): 10K, Resistor_SMD:R_0603_1608Metric_Pad0.98x0.95mm_HandSolder, symbol ISAAC-rescue:R_Small_US-Device
- added U? (x8): DMN4026SSD, footprints:SOIC127P600X150-8N, symbol New_Library:DMN4026SSD
- D?: footprint (none) -> Diode_SMD:D_1812_4532Metric_Pad1.30x3.40mm_HandSolder; symbol pspice:DIODE -> ISAAC-rescue:DIODE-pspice
- R?: footprint (none) -> Resistor_SMD:R_0603_1608Metric_Pad0.98x0.95mm_HandSolder; symbol Device:R_Small_US -> ISAAC-rescue:R_Small_US-Device
Connections:
- net labels added: GATE10, GATE11, GATE12, GATE13, GATE14, GATE15, GATE16, GATE2, GATE3, GATE4, GATE5, GATE6, GATE7, GATE8, GATE9, GND, SOL10, SOL11, SOL12, SOL13, SOL14, SOL15, SOL16, SOL2, SOL3, SOL4, SOL5, SOL6, SOL7, SOL8, SOL9, VCC
- wire segments 6 -> 212

Commit message: Added Pico, Molex Connectors, MPU6050
Parts:
- removed J? (x2): Screw_Terminal_01x08, TerminalBlock_TE-Connectivity:TerminalBlock_TE_282834-8_1x08_P2.54mm_Horizontal, symbol Connector:Screw_Terminal_01x08
- added C?: C_Small, symbol Device:C_Small
- added C?: CP1_Small, symbol Device:CP1_Small
- added J? (x2): Conn_02x04_Top_Bottom, Connector_Molex:Molex_Mini-Fit_Jr_5569-08A2_2x04_P4.20mm_Horizontal, symbol Connector_Generic:Conn_02x04_Top_Bottom
- added U?: Pico, RPi_Pico:RPi_Pico_SMD_TH, symbol MCU_RaspberryPi_and_Boards:Pico
- added U?: module_mpu6050, usini_sensors:module_mpu6050, symbol usini_sensors:module_mpu6050
- added U?: LM337_TO3, Package_TO_SOT_THT:TO-3, symbol Regulator_Linear:LM337_TO3
- R? (x16): footprint Resistor_SMD:R_0603_1608Metric_Pad0.98x0.95mm_HandSolder -> Resistor_SMD:R_0805_2012Metric_Pad1.20x1.40mm_HandSolder
Connections:
- net labels added: +3.3V, +3.3VA, MPU_SCL, MPU_SDA
- wire segments 212 -> 227
Other:
- moved on the sheet: D?, R?, U?

Commit message: Added XT60 Conn and Started Tracing PCB
Parts:
- added J3: Screw_Terminal_01x02, footprints:TE_282837-2, symbol Connector:Screw_Terminal_01x02
- added J4: XT60PW-M, footprints:AMASS_XT60PW-M, symbol XT60PW-M:XT60PW-M
- C1, C2: renamed from C?; footprint (none) -> Capacitor_THT:CP_Radial_D4.0mm_P1.50mm
- U11: renamed from U?; footprint Package_TO_SOT_THT:TO-3 -> footprints:SOT230P696X180-4N
- e1: renamed from U?; footprint RPi_Pico:RPi_Pico_SMD_TH -> footprints:RPi_Pico_SMD_TH
- gave numbers to parts that had none: 43
Connections:
- net labels added: +BATT
- wire segments 227 -> 246
- no-connect marks 0 -> 26
Other:
- moved on the sheet: C1, C2, U11

Commit message: Finished Version 1
Parts:
- added H1, H2, H3, H4: MountingHole, MountingHole:MountingHole_3.2mm_M3, symbol Mechanical:MountingHole
Connections:
- net labels removed: +BATT
Changed lines of the file:
@@
 F 3 "~" H 7150 2325 50  0001 C CNN
 	1    7150 2325
-	0    1    1    0
+	1    0    0    -1
 $EndComp
 $Comp
@@
 Wire Wire Line
 	8600 5650 8500 5650
-$Comp
-L power:+BATT #PWR040
-U 1 1 61A49ECE
-P 8825 5650
-F 0 "#PWR040" H 8825 5500 50  0001 C CNN
-F 1 "+BATT" V 8840 5778 50  0000 L CNN
-F 2 "" H 8825 5650 50  0001 C CNN
-F 3 "" H 8825 5650 50  0001 C CNN
-	1    8825 5650
-	0    1    1    0
-$EndComp
 Wire Wire Line
 	8600 5650 8825 5650
@@
 	1    0    0    -1
 $EndComp
-$Comp
-L power:+BATT #PWR041
-U 1 1 61AB2293
-P 9875 5750
-F 0 "#PWR041" H 9875 5600 50  0001 C CNN
-F 1 "+BATT" V 9890 5877 50  0000 L CNN
-F 2 "" H 9875 5750 50  0001 C CNN
-F 3 "" H 9875 5750 50  0001 C CNN
-	1    9875 5750
-	0    -1   -1   0
-$EndComp
 Wire Wire Line
 	9875 5850 10075 5850
@@
 Wire Wire Line
 	1600 7125 1750 7125
-$Comp
-L power:+BATT #PWR043
-U 1 1 61C0B67A
-P 9975 3725
-F 0 "#PWR043" H 9975 3575 50  0001 C CNN
-F 1 "+BATT" V 9990 3853 50  0000 L CNN
-F 2 "" H 9975 3725 50  0001 C CNN
-F 3 "" H 9975 3725 50  0001 C CNN
-	1    9975 3725
-	0    1    1    0
-$EndComp
 Wire Wire Line
 	9725 3725 9975 3725
@@
 	1    9525 3825
 	-1   0    0    1
-$EndComp
-$Comp
-L power:+BATT #PWR044
-U 1 1 61C399E7
-P 9975 3825
-F 0 "#PWR044" H 9975 3675 50  0001 C CNN
-F 1 "+BATT" V 9990 3953 50  0000 L CNN
-F 2 "" H 9975 3825 50  0001 C CNN
-F 3 "" H 9975 3825 50  0001 C CNN
-	1    9975 3825
-	0    1    1    0
 $EndComp
 Wire Wire Line
@@
 Wire Wire Line
 	2850 3925 3150 3925
+$Comp
+L power:VCC #PWR0101
+U 1 1 625DCEF9
+P 9875 5750
+F 0 "#PWR0101" H 9875 5600 50  0001 C CNN
+F 1 "VCC" V 9890 5878 50  0000 L CNN
+F 2 "" H 9875 5750 50  0001 C CNN
+F 3 "" H 9875 5750 50  0001 C CNN
+	1    9875 5750
+	0    -1   -1   0
+$EndComp
+$Comp
+L power:VCC #PWR0102
+U 1 1 625DE706
+P 8825 5650
+F 0 "#PWR0102" H 8825 5500 50  0001 C CNN
+F 1 "VCC" V 8840 5778 50  0000 L CNN
+F 2 "" H 8825 5650 50  0001 C CNN
+F 3 "" H 8825 5650 50  0001 C CNN
+	1    8825 5650
+	0    1    1    0
+$EndComp
+$Comp
+L power:VCC #PWR0103
+U 1 1 625F6F3A
+P 9975 3825
+F 0 "#PWR0103" H 9975 3675 50  0001 C CNN
+F 1 "VCC" V 9990 3953 50  0000 L CNN
+F 2 "" H 9975 3825 50  0001 C CNN
+F 3 "" H 9975 3825 50  0001 C CNN
+	1    9975 3825
+	0    1    1    0
+$EndComp
+$Comp
+L power:VCC #PWR0104
+U 1 1 62624C30
+P 9975 3725
+F 0 "#PWR0104" H 9975 3575 50  0001 C CNN
+F 1 "VCC" V 9990 3853 50  0000 L CNN
+F 2 "" H 9975 3725 50  0001 C CNN
+F 3 "" H 9975 3725 50  0001 C CNN
+	1    9975 3725
+	0    1    1    0
+$EndComp
+$Comp
+L Mechanical:MountingHole H1
+U 1 1 6265BDBA
+P 10325 4550
+F 0 "H1" H 10425 4596 50  0000 L CNN
+F 1 "MountingHole" H 10425 4505 50  0000 L CNN
+F 2 "MountingHole:MountingHole_3.2mm_M3" H 10325 4550 50  0001 C CNN
+F 3 "~" H 10325 4550 50  0001 C CNN
+	1    10325 4550
+	1    0    0    -1
+$EndComp
+$Comp
+L Mechanical:MountingHole H2
+U 1 1 6265C573
+P 10325 4775
+F 0 "H2" H 10425 4821 50  0000 L CNN
+F 1 "MountingHole" H 10425 4730 50  0000 L CNN
+F 2 "MountingHole:MountingHole_3.2mm_M3" H 10325 4775 50  0001 C CNN
+F 3 "~" H 10325 4775 50  0001 C CNN
+	1    10325 4775
+	1    0    0    -1
+$EndComp
+$Comp
+L Mechanical:MountingHole H3
+U 1 1 6265CC0F
+P 10325 5000
+F 0 "H3" H 10425 5046 50  0000 L CNN
+F 1 "MountingHole" H 10425 4955 50  0000 L CNN
+F 2 "MountingHole:MountingHole_3.2mm_M3" H 10325 5000 50  0001 C CNN
+F 3 "~" H 10325 5000 50  0001 C CNN
+	1    10325 5000
+	1    0    0    -1
+$EndComp
+$Comp
+L Mechanical:MountingHole H4
+U 1 1 6265D090
+P 10325 5200
+F 0 "H4" H 10425 5246 50  0000 L CNN
+F 1 "MountingHole" H 10425 5155 50  0000 L CNN
+F 2 "MountingHole:MountingHole_3.2mm_M3" H 10325 5200 50  0001 C CNN
+F 3 "~" H 10325 5200 50  0001 C CNN
+	1    10325 5200
+	1    0    0    -1
+$EndComp
 $EndSCHEMATC

Commit message: Updated everything!
Parts:
- U10, U2, U3, U4, U5, U7, U8, U9: symbol New_Library:DMN4026SSD -> ISAAC-rescue:DMN4026SSD-New_Library
Connections:
- net GATE1: now also U2.6 (G1); no longer U2.2 (G1)
- net GATE10: now also U7.8 (G2); no longer U7.4 (G2)
- net GATE11: now also U8.6 (G1); no longer U8.2 (G1)
- net GATE12: now also U8.8 (G2); no longer U8.4 (G2)
- net GATE13: now also U9.6 (G1); no longer U9.2 (G1)
- net GATE14: now also U9.8 (G2); no longer U9.4 (G2)
- net GATE15: now also U10.6 (G1); no longer U10.2 (G1)
- net GATE16: now also U10.8 (G2); no longer U10.4 (G2)
- net GATE2: now also U2.8 (G2); no longer U2.4 (G2)
- net GATE3: now also U3.6 (G1); no longer U3.2 (G1)
- net GATE4: now also U3.8 (G2); no longer U3.4 (G2)
- net GATE5: now also U4.6 (G1); no longer U4.2 (G1)
- net GATE6: now also U4.8 (G2); no longer U4.4 (G2)
- net GATE7: now also U5.6 (G1); no longer U5.2 (G1)
- net GATE8: now also U5.8 (G2); no longer U5.4 (G2)
- net GATE9: now also U7.6 (G1); no longer U7.2 (G1)
- net SOL1: now also U2.5 (S1); no longer U2.1 (S1)
- net SOL10: now also U7.7 (S2); no longer U7.3 (S2)
- net SOL11: now also U8.5 (S1); no longer U8.1 (S1)
- net SOL12: now also U8.7 (S2); no longer U8.3 (S2)
- net SOL13: now also U9.5 (S1); no longer U9.1 (S1)
- net SOL14: now also U9.7 (S2); no longer U9.3 (S2)
- net SOL15: now also U10.5 (S1); no longer U10.1 (S1)
- net SOL16: now also U10.7 (S2); no longer U10.3 (S2)
- net SOL2: now also U2.7 (S2); no longer U2.3 (S2)
- net SOL3: now also U3.5 (S1); no longer U3.1 (S1)
- net SOL4: now also U3.7 (S2); no longer U3.3 (S2)
- net SOL5: now also U4.5 (S1); no longer U4.1 (S1)
- net SOL6: now also U4.7 (S2); no longer U4.3 (S2)
- net SOL7: now also U5.5 (S1); no longer U5.1 (S1)
- net SOL8: now also U5.7 (S2); no longer U5.3 (S2)
- net SOL9: now also U7.5 (S1); no longer U7.1 (S1)
- new net: D1.1 (K), U2.1 (D1), U2.2 (D1)
- new net: D2.1 (K), U2.3 (D2), U2.4 (D2)
- new net: D4.1 (K), U3.3 (D2), U3.4 (D2)
- new net: D3.1 (K), U3.1 (D1), U3.2 (D1)
- new net: D6.1 (K), U4.3 (D2), U4.4 (D2)
- new net: D5.1 (K), U4.1 (D1), U4.2 (D1)
- new net: D8.1 (K), U5.3 (D2), U5.4 (D2)
- new net: D7.1 (K), U5.1 (D1), U5.2 (D1)
- new net: D10.1 (K), U7.3 (D2), U7.4 (D2)
- new net: D9.1 (K), U7.1 (D1), U7.2 (D1)
- new net: D12.1 (K), U8.3 (D2), U8.4 (D2)
- new net: D11.1 (K), U8.1 (D1), U8.2 (D1)
- new net: D14.1 (K), U9.3 (D2), U9.4 (D2)
- new net: D13.1 (K), U9.1 (D1), U9.2 (D1)
- new net: D16.1 (K), U10.3 (D2), U10.4 (D2)
- new net: D15.1 (K), U10.1 (D1), U10.2 (D1)
Changed lines of the file:
@@
 GATE1
 $Comp
-L New_Library:DMN4026SSD U2
+L ISAAC-rescue:DMN4026SSD-New_Library U2
 U 1 1 616BD976
 P 2500 1325
@@
 GATE3
 $Comp
-L New_Library:DMN4026SSD U3
+L ISAAC-rescue:DMN4026SSD-New_Library U3
 U 1 1 6171067C
 P 2500 2325
@@
 GATE5
 $Comp
-L New_Library:DMN4026SSD U4
+L ISAAC-rescue:DMN4026SSD-New_Library U4
 U 1 1 61716C15
 P 2500 3325
@@
 GATE7
 $Comp
-L New_Library:DMN4026SSD U5
+L ISAAC-rescue:DMN4026SSD-New_Library U5
 U 1 1 6171B38E
 P 2500 4325
@@
 GATE9
 $Comp
-L New_Library:DMN4026SSD U7
+L ISAAC-rescue:DMN4026SSD-New_Library U7
 U 1 1 61730CEE
 P 6200 1325
@@
 GATE11
 $Comp
-L New_Library:DMN4026SSD U8
+L ISAAC-rescue:DMN4026SSD-New_Library U8
 U 1 1 6173F917
 P 6200 2275
@@
 GATE13
 $Comp
-L New_Library:DMN4026SSD U9
+L ISAAC-rescue:DMN4026SSD-New_Library U9
 U 1 1 6178B13B
 P 6200 3275
@@
 GATE15
 $Comp
-L New_Library:DMN4026SSD U10
+L ISAAC-rescue:DMN4026SSD-New_Library U10
 U 1 1 6179A8D8
 P 6200 4325
