File: ISAAC_PCB/ISAAC_V2.sch (KiCad schematic (older format))
At the start: 53 parts, among them J1 Conn_02x04_Top_Bottom, J2 Conn_02x04_Top_Bottom, J3 Screw_Terminal_01x02, J4 XT60PW-M, U10 DMN4026SSD, U11 LM337_TO3, U2 DMN4026SSD, U3 DMN4026SSD, U4 DMN4026SSD, U5 DMN4026SSD, U6 module_mpu6050, U7 DMN4026SSD, U8 DMN4026SSD, U9 DMN4026SSD

Commit message: Updated PCB and Tracing
Parts:
- U1: renamed from U?; footprint RPi_Pico:RPi_Pico_SMD_TH -> footprints:RPi_Pico_SMD_TH
Connections:
- net GND: now also J3.1 (Pin_1)
- net VCC: no longer J3.1 (Pin_1)
Changed lines of the file:
@@
-$EndComp
-$Comp
-L power:VCC #PWR0103
-U 1 1 625F6F3A
-P 9975 3825
-F 0 "#PWR0103" H 9975 3675 50  0001 C CNN
-F 1 "VCC" V 9990 3953 50  0000 L CNN
-F 2 "" H 9975 3825 50  0001 C CNN
-F 3 "" H 9975 3825 50  0001 C CNN
-	1    9975 3825
-	0    1    1    0
 $EndComp
 $Comp
@@
 	1650 4225 2250 4225
 $Comp
-L MCU_RaspberryPi_and_Boards:Pico U?
+L MCU_RaspberryPi_and_Boards:Pico U1
 U 1 1 6181702C
 P 2450 6175
-F 0 "U?" H 2450 7390 50  0000 C CNN
+F 0 "U1" H 2450 7390 50  0000 C CNN
 F 1 "Pico" H 2450 7299 50  0000 C CNN
-F 2 "RPi_Pico:RPi_Pico_SMD_TH" V 2450 6175 50  0001 C CNN
+F 2 "footprints:RPi_Pico_SMD_TH" V 2450 6175 50  0001 C CNN
 F 3 "" H 2450 6175 50  0001 C CNN
 	1    2450 6175
 	1    0    0    -1
 $EndComp
+$Comp
+L power:GND #PWR?
+U 1 1 61AD8BD8
+P 9975 3825
+F 0 "#PWR?" H 9975 3575 50  0001 C CNN
+F 1 "GND" V 9980 3697 50  0000 R CNN
+F 2 "" H 9975 3825 50  0001 C CNN
+F 3 "" H 9975 3825 50  0001 C CNN
+	1    9975 3825
+	0    -1   -1   0
+$EndComp
 $EndSCHEMATC
