File: ISAAC_PCB/ISAAC_V3.sch (KiCad schematic (older format))
At the start: 53 parts, among them J1 Conn_02x04_Top_Bottom, J2 Conn_02x04_Top_Bottom, J3 Screw_Terminal_01x02, J4 XT60PW-M, U10 DMN4026SSD, U11 LM337_TO3, U2 DMN4026SSD, U3 DMN4026SSD, U4 DMN4026SSD, U5 DMN4026SSD, U6 module_mpu6050, U7 DMN4026SSD, U8 DMN4026SSD, U9 DMN4026SSD

Commit message: Updated PCB and Tracing
Parts:
- removed U?: Pico, RPi_Pico:RPi_Pico_SMD_TH, symbol MCU_RaspberryPi_and_Boards:Pico
Connections:
- net GND: now also J3.1 (Pin_1)
- net VCC: no longer J3.1 (Pin_1)
- no-connect marks 41 -> 19
Changed lines of the file:
@@
 Text GLabel 9250 2075 0    50   Input ~ 0
 SOL11
-Text GLabel 1250 5225 0    50   Input ~ 0
-GATE2
-Text GLabel 1250 5125 0    50   Input ~ 0
-GATE1
-Text GLabel 1250 6225 0    50   Input ~ 0
-GATE10
-Text GLabel 1250 6125 0    50   Input ~ 0
-GATE9
-Text GLabel 1250 6025 0    50   Input ~ 0
-GATE8
-Text GLabel 1250 5925 0    50   Input ~ 0
-GATE7
-Text GLabel 1250 5725 0    50   Input ~ 0
-GATE6
-Text GLabel 1250 5625 0    50   Input ~ 0
-GATE5
-Text GLabel 1250 5525 0    50   Input ~ 0
-GATE4
-Text GLabel 1250 5425 0    50   Input ~ 0
-GATE3
-Text GLabel 1250 6425 0    50   Input ~ 0
-GATE11
-Text GLabel 1250 6525 0    50   Input ~ 0
-GATE12
-Text GLabel 1250 6625 0    50   Input ~ 0
-GATE13
-Text GLabel 1250 6725 0    50   Input ~ 0
-GATE14
-Text GLabel 1250 6925 0    50   Input ~ 0
-GATE15
-Text GLabel 1250 7025 0    50   Input ~ 0
-GATE16
 Text GLabel 9275 3850 0    50   Input ~ 0
 MPU_SDA
-Text GLabel 3025 7025 2    50   Input ~ 0
-MPU_SDA
 Wire Wire Line
 	9275 3850 9575 3850
-Wire Wire Line
-	2800 7025 3025 7025
 $Comp
 L usini_sensors:module_mpu6050 U6
@@
 Wire Wire Line
 	9275 3750 9575 3750
-Text GLabel 3025 6925 2    50   Input ~ 0
-MPU_SCL
-Wire Wire Line
-	2800 6925 3025 6925
-$Comp
-L power:+3.3V #PWR09
-U 1 1 6195DE97
-P 2975 5525
-F 0 "#PWR09" H 2975 5375 50  0001 C CNN
-F 1 "+3.3V" V 2990 5653 50  0000 L CNN
-F 2 "" H 2975 5525 50  0001 C CNN
-F 3 "" H 2975 5525 50  0001 C CNN
-	1    2975 5525
-	0    1    1    0
-$EndComp
 $Comp
 L power:+3.3V #PWR020
@@
 $EndComp
 Wire Wire Line
-	2975 5525 2800 5525
-Wire Wire Line
 	9200 3550 9575 3550
 $Comp
@@
 Wire Wire Line
 	9200 3650 9575 3650
-$Comp
-L power:GND #PWR011
-U 1 1 6198DA00
-P 3000 5325
-F 0 "#PWR011" H 3000 5075 50  0001 C CNN
-F 1 "GND" V 3005 5197 50  0000 R CNN
-F 2 "" H 3000 5325 50  0001 C CNN
-F 3 "" H 3000 5325 50  0001 C CNN
-	1    3000 5325
-	0    -1   -1   0
-$EndComp
-Wire Wire Line
-	3000 5325 2800 5325
 $Comp
 L Regulator_Linear:LM337_TO3 U11
@@
 $EndComp
 Wire Wire Line
-	1250 5125 1400 5125
-Wire Wire Line
-	1400 5225 1250 5225
-Wire Wire Line
-	1250 5425 1400 5425
-Wire Wire Line
-	1400 5525 1250 5525
-Wire Wire Line
-	1250 5625 1400 5625
-Wire Wire Line
-	1250 5725 1400 5725
-Wire Wire Line
-	1250 5925 1400 5925
-Wire Wire Line
-	1400 6025 1250 6025
-Wire Wire Line
-	1250 6125 1400 6125
-Wire Wire Line
-	1400 6225 1250 6225
-Wire Wire Line
-	1250 6425 1400 6425
-Wire Wire Line
-	1400 6525 1250 6525
-Wire Wire Line
-	1250 6625 1400 6625
-Wire Wire Line
-	1250 6725 1400 6725
-Wire Wire Line
-	1400 6925 1250 6925
-Wire Wire Line
-	1250 7025 1400 7025
-Wire Wire Line
 	9750 2900 10000 2900
 $Comp
@@
 Wire Wire Line
 	10000 3000 9750 3000
-$Comp
-L power:+3.3VA #PWR010
-U 1 1 61C4EC19
-P 3000 5225
-F 0 "#PWR010" H 3000 5075 50  0001 C CNN
-F 1 "+3.3VA" V 3015 5352 50  0000 L CNN
-F 2 "" H 3000 5225 50  0001 C CNN
-F 3 "" H 3000 5225 50  0001 C CNN
-	1    3000 5225
-	0    1    1    0
-$EndComp
-Wire Wire Line
-	3000 5225 2800 5225
-NoConn ~ 1400 6825
-NoConn ~ 1400 6325
-NoConn ~ 1400 5825
-NoConn ~ 1400 5325
-NoConn ~ 2800 5125
-NoConn ~ 2800 5425
-NoConn ~ 2800 5625
-NoConn ~ 2800 5725
-NoConn ~ 2800 5825
-NoConn ~ 2800 5925
-NoConn ~ 2800 6025
-NoConn ~ 2800 6125
-NoConn ~ 2800 6225
-NoConn ~ 2800 6325
-NoConn ~ 2800 6425
-NoConn ~ 2800 6525
-NoConn ~ 2800 6625
-NoConn ~ 2800 6725
-NoConn ~ 2800 6825
-NoConn ~ 2200 7225
-NoConn ~ 2100 7225
-NoConn ~ 2000 7225
 NoConn ~ 9575 4250
 NoConn ~ 9575 4150
@@
 $EndComp
 $Comp
-L power:VCC #PWR0103
-U 1 1 625F6F3A
-P 10000 3000
-F 0 "#PWR0103" H 10000 2850 50  0001 C CNN
-F 1 "VCC" V 10015 3128 50  0000 L CNN
-F 2 "" H 10000 3000 50  0001 C CNN
-F 3 "" H 10000 3000 50  0001 C CNN
-	1    10000 3000
-	0    1    1    0
-$EndComp
-$Comp
 L power:VCC #PWR0104
 U 1 1 62624C30
@@
 Wire Wire Line
 	1650 4225 2250 4225
-$Comp
-L MCU_RaspberryPi_and_Boards:Pico U?
-U 1 1 6181702C
-P 2100 6075
-F 0 "U?" H 2100 7290 50  0000 C CNN
-F 1 "Pico" H 2100 7199 50  0000 C CNN
-F 2 "RPi_Pico:RPi_Pico_SMD_TH" V 2100 6075 50  0001 C CNN
-F 3 "" H 2100 6075 50  0001 C CNN
-	1    2100 6075
-	1    0    0    -1
-$EndComp
 $Sheet
 S 4025 4975 2350 2650
@@
 Text Notes 9825 5600 0    118  ~ 24
 XT60 PWR In\n
+$Comp
+L power:GND #PWR0103
+U 1 1 618DC8F5
+P 10000 3000
+F 0 "#PWR0103" H 10000 2750 50  0001 C CNN
+F 1 "GND" V 10005 2872 50  0000 R CNN
+F 2 "" H 10000 3000 50  0001 C CNN
+F 3 "" H 10000 3000 50  0001 C CNN
+	1    10000 3000
+	0    -1   -1   0
+$EndComp
 $EndSCHEMATC
