File: ISAAC_PCB/rp2040_min_req.sch (KiCad schematic (older format))
At the start: 25 parts

Commit message: Updated PCB and Tracing
Parts:
- gave numbers to parts that had none: 25
Connections:
- net +3V3: no longer C10.1, C11.1, C12.1, C17.1, C4.1, C5.1, C6.1, C7.1, C8.1, C9.1, U12.1 (IOVDD), U12.10 (IOVDD), U12.22 (IOVDD), U12.33 (IOVDD), U12.42 (IOVDD), U12.43 (ADC_AVDD), U12.44 (VREG_IN), U12.48 (USB_VDD), U12.49 (IOVDD), U13.2 (VO)
- new net +3.3VA: C10.1, C11.1, C12.1, C17.1, C4.1, C5.1, C6.1, C7.1, C8.1, C9.1, U12.1 (IOVDD), U12.10 (IOVDD), U12.22 (IOVDD), U12.33 (IOVDD), U12.42 (IOVDD), U12.43 (ADC_AVDD), U12.44 (VREG_IN), U12.48 (USB_VDD), U12.49 (IOVDD), U13.2 (VO)
